Commit message: clean up _odom_to_tf

File: dimos/robot/unitree/go2/go2.urdf (robot description, URDF)
Before this commit: robot go2, 3 links, 2 joints
Links:
- added link lidar_link
Joints:
- added joint base_link_to_lidar_link: type fixed, parent base_link, child lidar_link, origin xyz=0.0 0.0 0.0 rpy=0 0 0
