Commit message: small china corrections

File: dimos/robot/unitree/g1/g1.urdf (robot description, URDF)
Before this commit: robot g1_29dof_rev_1_0, 40 links, 39 joints
Joints:
- joint mid360_joint: origin xyz=0.0002835 0.00003 0.41618 rpy=0 0.04014257279586953 0 -> xyz=0.0002835 0.00003 0.41618 rpy=0 -0.04014257279586953 0
