Commit message: Revert "fix(g1): mid360_joint carries the real upside-down mount (roll pi)"
This reverts commit 8c61278d059584b8922efe9e2a622b4efec11d40.

File: dimos/robot/unitree/g1/g1.urdf (robot description, URDF)
Before this commit: robot g1_29dof_rev_1_0, 40 links, 39 joints
Joints:
- joint mid360_joint: origin xyz=0.0002835 0.00003 0.41618 rpy=3.141592653589793 0.04014257279586953 0 -> xyz=0.0002835 0.00003 0.41618 rpy=0 0.04014257279586953 0
